Commit message: Add Ridgeback wheels to URDF.

File: urdf/xacro/thing.urdf.xacro (robot description, xacro)
@@ -1,212 +1,5 @@
-<?xml version="1.0" encoding="utf-8"?>
-<robot name="Thing" xmlns:xacro="http://wiki.ros.org/xacro">
-  <material name="dark_grey">
-    <color rgba="0.2 0.2 0.2 1.0"/>
-  </material>
-  <material name="light_grey">
-    <color rgba="0.4 0.4 0.4 1.0"/>
-  </material>
-  <material name="red">
-    <color rgba="0.8 0.0 0.0 1.0"/>
-  </material>
-  <material name="white">
-    <color rgba="0.9 0.9 0.9 1.0"/>
-  </material>
-  <material name="yellow">
-    <color rgba="0.8 0.8 0.0 1.0"/>
-  </material>
-  <material name="black">
-    <color rgba="0.15 0.15 0.15 1.0"/>
-  </material>
-  <material name="seethrough">
-    <color rgba="1.0 0.0 0.0 0.25"/>
-  </material>
-  <link name="base_link">
-	 <inertial>
-     <mass value="0.01"/>
-     <inertia ixx="0.01" ixy="0" ixz="0" iyy="0.01" iyz="0" izz="0.01"/>
-     <origin rpy="0 0 0" xyz="0 0 0"/>
-    </inertial>
-  </link>
-  <joint name="base_link_joint" type="fixed">
-    <origin rpy="0 0 0" xyz="0 0 0"/>
-    <parent link="base_link"/>
-    <child link="chassis_link"/>
-  </joint>
-  <link name="chassis_link">
-    <visual>
-      <geometry>
-        <mesh filename="file://$(find upright_assets)/thing/meshes/ridgeback/body.stl"/>
-      </geometry>
-      <material name="black"/>
-    </visual>
-    <collision>
-      <origin xyz="0 0 0"/>
-      <geometry>
-        <mesh filename="file://$(find upright_assets)/thing/meshes/ridgeback/body-collision.stl"/>
-      </geometry>
-    </collision>
-    <inertial>
-      <origin rpy="1.57079632679 0 1.57079632679" xyz="0.012 0.002 0.067"/>
-      <!-- <origin rpy="1.57079632679 0 1.57079632679" xyz="0 0 0"/> -->
-      <mass value="165.304"/>
-      <inertia ixx="4.4744" ixy="0.03098" ixz="0.003647" iyy="7.1624" iyz="0.1228" izz="4.6155"/>
-    </inertial>
-  </link>
-  <joint name="right_side_cover_link_joint" type="fixed">
-    <origin rpy="0 0 0" xyz="0 0 0"/>
-    <parent link="chassis_link"/>
-    <child link="right_side_cover_link"/>
-  </joint>
-  <joint name="left_side_cover_link_joint" type="fixed">
-    <origin rpy="0 0 0" xyz="0 0 0"/>
-    <parent link="chassis_link"/>
-    <child link="left_side_cover_link"/>
-  </joint>
-  <link name="left_side_cover_link">
-    <visual>
-      <origin rpy="0 0 3.14159265359" xyz="0 0 0"/>
-      <geometry>
-        <mesh filename="file://$(find upright_assets)/thing/meshes/ridgeback/side-cover.stl"/>
-      </geometry>
-      <material name="yellow"/>
-    </visual>
-  </link>
-  <link name="right_side_cover_link">
-    <visual>
-      <origin rpy="0 0 0" xyz="0 0 0"/>
-      <geometry>
-        <mesh filename="file://$(find upright_assets)/thing/meshes/ridgeback/side-cover.stl"/>
-      </geometry>
-      <material name="yellow"/>
-    </visual>
-  </link>
-  <joint name="front_cover_link_joint" type="fixed">
-    <origin rpy="0 0 0" xyz="0 0 0"/>
-    <parent link="chassis_link"/>
-    <child link="front_cover_link"/>
-  </joint>
-  <link name="front_cover_link">
-    <visual>
-      <origin rpy="0 0 0" xyz="0 0 0"/>
-      <geometry>
-        <mesh filename="file://$(find upright_assets)/thing/meshes/ridgeback/end-cover.stl"/>
-      </geometry>
-      <material name="black"/>
-    </visual>
-  </link>
-  <joint name="rear_cover_link_joint" type="fixed">
-    <origin rpy="0 0 0" xyz="0 0 0"/>
-    <parent link="chassis_link"/>
-    <child link="rear_cover_link"/>
-  </joint>
-  <link name="rear_cover_link">
-    <visual>
-      <origin rpy="0 0 3.14159265359" xyz="0 0 0"/>
-      <geometry>
-        <mesh filename="file://$(find upright_assets)/thing/meshes/ridgeback/end-cover.stl"/>
-      </geometry>
-      <material name="black"/>
-    </visual>
-  </link>
-  <joint name="front_lights_link_joint" type="fixed">
-    <origin rpy="0 0 0" xyz="0 0 0"/>
-    <parent link="chassis_link"/>
-    <child link="front_lights_link"/>
-  </joint>
-  <joint name="rear_lights_link_joint" type="fixed">
-    <origin rpy="0 0 0" xyz="0 0 0"/>
-    <parent link="chassis_link"/>
-    <child link="rear_lights_link"/>
-  </joint>
-  <link name="front_lights_link">
-    <visual>
-      <origin rpy="0 0 0" xyz="0 0 0"/>
-      <geometry>
-        <mesh filename="file://$(find upright_assets)/thing/meshes/ridgeback/lights.stl"/>
-      </geometry>
-      <material name="white"/>
-    </visual>
-  </link>
-  <link name="rear_lights_link">
-    <visual>
-      <origin rpy="0 0 3.14159265359" xyz="0 0 0"/>
-      <geometry>
-        <mesh filename="file://$(find upright_assets)/thing/meshes/ridgeback/lights.stl"/>
-      </geometry>
-      <material name="red"/>
-    </visual>
-  </link>
-  <joint name="top_link_joint" type="fixed">
-    <origin rpy="0 0 0" xyz="0 0 0"/>
-    <parent link="chassis_link"/>
-    <child link="top_link"/>
-  </joint>
-  <link name="top_link">
-    <visual>
-      <origin rpy="0 0 0" xyz="0 0 0"/>
-      <geometry>
-        <mesh filename="file://$(find upright_assets)/thing/meshes/ridgeback/top.stl"/>
-      </geometry>
-      <material name="black"/>
-    </visual>
-    <collision>
-      <origin rpy="0 0 0" xyz="0 0 0"/>
-      <geometry>
-        <mesh filename="file://$(find upright_assets)/thing/meshes/ridgeback/top.stl"/>
-      </geometry>
-    </collision>
-  </link>
-  <link name="arch_link">
-    <visual>
-      <geometry>
-        <mesh filename="file://$(find upright_assets)/thing/meshes/tor11_mech.dae"/>
-      </geometry>
-      <material name="LightGrey">
-        <color rgba="0.7 0.7 0.7 1.0"/>
-      </material>
-    </visual>
-  </link>
-  <joint name="arch_joint" type="fixed">
-    <origin rpy="0 0 1.57079632679" xyz="0 0 0.278"/>
-    <!-- <origin rpy="-1.57079632679 0 1.57079632679" xyz="0 0 0.278"/> -->
-    <parent link="top_link"/>
-    <child link="arch_link"/>
-  </joint>
-  <!-- UR10 arm -->
-  <xacro:include filename="$(find ur_description)/urdf/inc/ur10_macro.xacro"/>
-  <xacro:ur10_robot
-    prefix="ur10_arm_"
-    visual_parameters_file="$(find upright_assets)/config/ur10/visual_parameters.yaml"
-    kinematics_parameters_file="$(find upright_assets)/config/ur10/calibration.yaml"
-  />
-  <!-- Join arm to the base -->
-  <joint name="ur10_arm_base" type="fixed">
-    <parent link="arch_link"/>
-    <child link="ur10_arm_base_link"/>
-    <origin rpy="0.0 0.0 3.14159265359" xyz="0.01 -0.27 0.375"/>
-  </joint>
-  <!-- Frame coincident with all-zeros TCP on UR controller -->
-  <link name="gripper">
-    <visual>
-      <!-- start halfway along the cylinder -->
-      <origin rpy="0 0 0" xyz="0 0 0.145"/>
-      <geometry>
-        <cylinder length="0.290" radius="0.01"/>
-      </geometry>
-      <material name="black"/>
-    </visual>
-    <collision>
-      <origin rpy="0 0 0" xyz="0 0 0.145"/>
-      <geometry>
-        <cylinder length="0.290" radius="0.01"/>
-      </geometry>
-    </collision>
-  </link>
-  <joint name="tool_gripper_joint" type="fixed">
-    <!-- The 15-degree offset about the z-axis is to account for the fact that the gripper is actually mounted at this offset. -->
-    <origin rpy="0 0 0.2617993877991494" xyz="0 0.0 0"/>
-    <parent link="ur10_arm_tool0"/>
-    <child link="gripper"/>
-  </joint>
+<?xml version="1.0" ?>
+<robot name="mm_ocs2_tray" xmlns:xacro="http://www.ros.org/wiki/xacro">
+  <xacro:include filename="ridgeback_wheels.urdf.xacro" />
+  <xacro:include filename="thing_no_wheels.urdf.xacro" />
 </robot>
