Commit message: Add meshes, move some ROS utilities to separate library.

File: urdf/xacro/ridgeback_wheels.urdf.xacro (robot description, xacro)
@@ -20,5 +20,5 @@
         <origin xyz="0 0 0" rpy="${PI/2} 0 0"/>
         <geometry>
-          <mesh filename="file://$(find upright_assets)/thing/meshes/ridgeback/wheel.stl"/>
+          <mesh filename="file://$(find mobile_manipulation_central)/meshes/ridgeback/wheel.stl"/>
         </geometry>
         <material name="black" />
@@ -60,5 +60,5 @@
         <origin xyz="0 0 0" rpy="${PI/2} 0 ${PI/2}" />
         <geometry>
-          <mesh filename="file://$(find upright_assets)/thing/meshes/ridgeback/rocker.stl"/>
+          <mesh filename="file://$(find mobile_manipulation_central)/meshes/ridgeback/rocker.stl"/>
         </geometry>
         <material name="black" />
@@ -103,5 +103,5 @@
       <origin xyz="0 0 0" rpy="0 ${PI/2} 0" />
       <geometry>
-        <mesh filename="file://$(find upright_assets)/thing/meshes/ridgeback/axle.stl" />
+        <mesh filename="file://$(find mobile_manipulation_central)/meshes/ridgeback/axle.stl" />
       </geometry>
       <material name="black" />

File: urdf/xacro/thing_no_wheels.urdf.xacro (robot description, xacro)
@@ -45,5 +45,5 @@
     <visual>
       <geometry>
-        <mesh filename="file://$(find upright_assets)/thing/meshes/ridgeback/body.stl"/>
+        <mesh filename="file://$(find mobile_manipulation_central)/meshes/ridgeback/body.stl"/>
       </geometry>
       <material name="black"/>
@@ -52,5 +52,5 @@
       <origin xyz="0 0 0"/>
       <geometry>
-        <mesh filename="file://$(find upright_assets)/thing/meshes/ridgeback/body-collision.stl"/>
+        <mesh filename="file://$(find mobile_manipulation_central)/meshes/ridgeback/body-collision.stl"/>
       </geometry>
     </collision>
@@ -76,5 +76,5 @@
       <origin rpy="0 0 3.14159265359" xyz="0 0 0"/>
       <geometry>
-        <mesh filename="file://$(find upright_assets)/thing/meshes/ridgeback/side-cover.stl"/>
+        <mesh filename="file://$(find mobile_manipulation_central)/meshes/ridgeback/side-cover.stl"/>
       </geometry>
       <material name="yellow"/>
@@ -85,5 +85,5 @@
       <origin rpy="0 0 0" xyz="0 0 0"/>
       <geometry>
-        <mesh filename="file://$(find upright_assets)/thing/meshes/ridgeback/side-cover.stl"/>
+        <mesh filename="file://$(find mobile_manipulation_central)/meshes/ridgeback/side-cover.stl"/>
       </geometry>
       <material name="yellow"/>
@@ -99,5 +99,5 @@
       <origin rpy="0 0 0" xyz="0 0 0"/>
       <geometry>
-        <mesh filename="file://$(find upright_assets)/thing/meshes/ridgeback/end-cover.stl"/>
+        <mesh filename="file://$(find mobile_manipulation_central)/meshes/ridgeback/end-cover.stl"/>
       </geometry>
       <material name="black"/>
@@ -113,5 +113,5 @@
       <origin rpy="0 0 3.14159265359" xyz="0 0 0"/>
       <geometry>
-        <mesh filename="file://$(find upright_assets)/thing/meshes/ridgeback/end-cover.stl"/>
+        <mesh filename="file://$(find mobile_manipulation_central)/meshes/ridgeback/end-cover.stl"/>
       </geometry>
       <material name="black"/>
@@ -132,5 +132,5 @@
       <origin rpy="0 0 0" xyz="0 0 0"/>
       <geometry>
-        <mesh filename="file://$(find upright_assets)/thing/meshes/ridgeback/lights.stl"/>
+        <mesh filename="file://$(find mobile_manipulation_central)/meshes/ridgeback/lights.stl"/>
       </geometry>
       <material name="white"/>
@@ -141,5 +141,5 @@
       <origin rpy="0 0 3.14159265359" xyz="0 0 0"/>
       <geometry>
-        <mesh filename="file://$(find upright_assets)/thing/meshes/ridgeback/lights.stl"/>
+        <mesh filename="file://$(find mobile_manipulation_central)/meshes/ridgeback/lights.stl"/>
       </geometry>
       <material name="red"/>
@@ -155,5 +155,5 @@
       <origin rpy="0 0 0" xyz="0 0 0"/>
       <geometry>
-        <mesh filename="file://$(find upright_assets)/thing/meshes/ridgeback/top.stl"/>
+        <mesh filename="file://$(find mobile_manipulation_central)/meshes/ridgeback/top.stl"/>
       </geometry>
       <material name="black"/>
@@ -162,5 +162,5 @@
       <origin rpy="0 0 0" xyz="0 0 0"/>
       <geometry>
-        <mesh filename="file://$(find upright_assets)/thing/meshes/ridgeback/top.stl"/>
+        <mesh filename="file://$(find mobile_manipulation_central)/meshes/ridgeback/top.stl"/>
       </geometry>
     </collision>
@@ -169,5 +169,5 @@
     <visual>
       <geometry>
-        <mesh filename="file://$(find upright_assets)/thing/meshes/tor11_mech.dae"/>
+        <mesh filename="file://$(find mobile_manipulation_central)/meshes/tor11_mech.dae"/>
       </geometry>
       <material name="LightGrey">
@@ -186,6 +186,6 @@
   <xacro:ur10_robot
     prefix="ur10_arm_"
-    visual_parameters_file="$(find upright_assets)/config/ur10/visual_parameters.yaml"
-    kinematics_parameters_file="$(find upright_assets)/config/ur10/calibration.yaml"
+    visual_parameters_file="$(find mobile_manipulation_central)/config/ur10/visual_parameters.yaml"
+    kinematics_parameters_file="$(find mobile_manipulation_central)/config/ur10/calibration.yaml"
   />
   <!-- Join arm to the base -->
