Commit message: Finish script to calibrate EE.

File: urdf/xacro/thing_no_wheels.urdf.xacro (robot description, xacro)
@@ -30,4 +30,6 @@
     <color rgba="1.0 0.0 0.0 0.25"/>
   </material>
+  <xacro:property name="transform_parameters_file" value="$(find mobile_manipulation_central)/config/ur10/transforms.yaml"/>
+  <xacro:property name="config_transform_parameters" value="${load_yaml(transform_parameters_file)}"/>
   <link name="base_link">
 	 <inertial>
@@ -37,6 +39,11 @@
     </inertial>
   </link>
+  <!-- <joint name="base_link_joint" type="fixed"> -->
+  <!--   <origin rpy="0 0 0" xyz="0 0 0"/> -->
+  <!--   <parent link="base_link"/> -->
+  <!--   <child link="chassis_link"/> -->
+  <!-- </joint> -->
   <joint name="base_link_joint" type="fixed">
-    <origin rpy="0 0 0" xyz="0 0 0"/>
+    <origin rpy="${config_transform_parameters['T1']['rpy'][0]} ${config_transform_parameters['T1']['rpy'][1]} ${config_transform_parameters['T1']['rpy'][2]}" xyz="${config_transform_parameters['T1']['xyz'][0]} ${config_transform_parameters['T1']['xyz'][1]} ${config_transform_parameters['T1']['xyz'][2]}"/>
     <parent link="base_link"/>
     <child link="chassis_link"/>
@@ -218,3 +225,10 @@
     <child link="gripper"/>
   </joint>
+  <!-- Extra link for the gripped object, which must be calibrated. -->
+  <link name="gripped_object" />
+  <joint name="gripped_object_joint" type="fixed">
+    <origin rpy="${config_transform_parameters['T2']['rpy'][0]} ${config_transform_parameters['T2']['rpy'][1]} ${config_transform_parameters['T2']['rpy'][2]}" xyz="${config_transform_parameters['T2']['xyz'][0]} ${config_transform_parameters['T2']['xyz'][1]} ${config_transform_parameters['T2']['xyz'][2]}"/>
+    <parent link="gripper"/>
+    <child link="gripped_object"/>
+  </joint>
 </robot>

Commit message: More elegantly and flexibly include calibration parameters in URDFs.
Works whether the URDF is being loaded into the ROS parameter server or
just being compiled with xacro elsewere.

File: urdf/xacro/thing_no_wheels.urdf.xacro (robot description, xacro)
@@ -30,6 +30,16 @@
     <color rgba="1.0 0.0 0.0 0.25"/>
   </material>
-  <xacro:property name="transform_parameters_file" value="$(find mobile_manipulation_central)/config/ur10/transforms.yaml"/>
-  <xacro:property name="config_transform_parameters" value="${load_yaml(transform_parameters_file)}"/>
+  <xacro:arg name="kinematics_params" default="$(find mobile_manipulation_central)/config/ur10/kinematics_parameters.yaml"/>
+  <xacro:arg name="visual_params" default="$(find mobile_manipulation_central)/config/ur10/visual_parameters.yaml"/>
+  <xacro:arg name="transform_params" default="$(find mobile_manipulation_central)/config/ur10/transforms.yaml"/>
+  <!-- Load the base and tool transforms -->
+  <xacro:property name="transform_params_file" value="$(arg transform_params)" />
+  <xacro:property name="config_transform_parameters" value="${load_yaml(transform_params_file)}"/>
+  <!-- Macro to use a transform from `config_transform_parameters` as the origin. -->
+  <xacro:macro name="transformed_origin" params="name">
+    <xacro:property name="T" value="${config_transform_parameters[name]}" />
+    <origin rpy="${T['rpy'][0]} ${T['rpy'][1]} ${T['rpy'][2]}"
+            xyz="${T['xyz'][0]} ${T['xyz'][1]} ${T['xyz'][2]}"/>
+  </xacro:macro>
   <link name="base_link">
 	 <inertial>
@@ -45,5 +55,5 @@
   <!-- </joint> -->
   <joint name="base_link_joint" type="fixed">
-    <origin rpy="${config_transform_parameters['T1']['rpy'][0]} ${config_transform_parameters['T1']['rpy'][1]} ${config_transform_parameters['T1']['rpy'][2]}" xyz="${config_transform_parameters['T1']['xyz'][0]} ${config_transform_parameters['T1']['xyz'][1]} ${config_transform_parameters['T1']['xyz'][2]}"/>
+    <xacro:transformed_origin name="T1" />
     <parent link="base_link"/>
     <child link="chassis_link"/>
@@ -193,6 +203,6 @@
   <xacro:ur10_robot
     prefix="ur10_arm_"
-    visual_parameters_file="$(find mobile_manipulation_central)/config/ur10/visual_parameters.yaml"
-    kinematics_parameters_file="$(find mobile_manipulation_central)/config/ur10/calibration.yaml"
+    visual_parameters_file="$(arg visual_params)"
+    kinematics_parameters_file="$(arg kinematics_params)"
   />
   <!-- Join arm to the base -->
@@ -228,5 +238,5 @@
   <link name="gripped_object" />
   <joint name="gripped_object_joint" type="fixed">
-    <origin rpy="${config_transform_parameters['T2']['rpy'][0]} ${config_transform_parameters['T2']['rpy'][1]} ${config_transform_parameters['T2']['rpy'][2]}" xyz="${config_transform_parameters['T2']['xyz'][0]} ${config_transform_parameters['T2']['xyz'][1]} ${config_transform_parameters['T2']['xyz'][2]}"/>
+    <xacro:transformed_origin name="T2" />
     <parent link="gripper"/>
     <child link="gripped_object"/>

Commit message: Make URDF somewhat more generic by getting rid of the gripped object.

File: urdf/xacro/thing_no_wheels.urdf.xacro (robot description, xacro)
@@ -235,10 +235,10 @@
     <child link="gripper"/>
   </joint>
-  <!-- Extra link for the gripped object, which must be calibrated. -->
-  <link name="gripped_object" />
-  <joint name="gripped_object_joint" type="fixed">
-    <xacro:transformed_origin name="T2" />
-    <parent link="gripper"/>
-    <child link="gripped_object"/>
-  </joint>
+  <!-- If you want to have an object as part of the URDF, include something like: -->
+  <!-- <link name="gripped_object" /> -->
+  <!-- <joint name="gripped_object_joint" type="fixed"> -->
+  <!--   <xacro:transformed_origin name="T2" /> -->
+  <!--   <parent link="gripper"/> -->
+  <!--   <child link="gripped_object"/> -->
+  <!-- </joint> -->
 </robot>

Commit message: Fix joint name collision.

File: urdf/xacro/thing_no_wheels.urdf.xacro (robot description, xacro)
@@ -207,5 +207,5 @@
   />
   <!-- Join arm to the base -->
-  <joint name="ur10_arm_base" type="fixed">
+  <joint name="ur10_arm_base_joint" type="fixed">
     <parent link="arch_link"/>
     <child link="ur10_arm_base_link"/>

Commit message: More descriptive names for calibrated transforms.

File: urdf/xacro/thing_no_wheels.urdf.xacro (robot description, xacro)
@@ -49,11 +49,7 @@
     </inertial>
   </link>
-  <!-- <joint name="base_link_joint" type="fixed"> -->
-  <!--   <origin rpy="0 0 0" xyz="0 0 0"/> -->
-  <!--   <parent link="base_link"/> -->
-  <!--   <child link="chassis_link"/> -->
-  <!-- </joint> -->
+  <!-- Transform between base and arm can be calibrated and is loaded from parameters. -->
   <joint name="base_link_joint" type="fixed">
-    <xacro:transformed_origin name="T1" />
+    <xacro:transformed_origin name="base_to_arm_transform" />
     <parent link="base_link"/>
     <child link="chassis_link"/>
@@ -238,5 +234,5 @@
   <!-- <link name="gripped_object" /> -->
   <!-- <joint name="gripped_object_joint" type="fixed"> -->
-  <!--   <xacro:transformed_origin name="T2" /> -->
+  <!--   <xacro:transformed_origin name="gripped_object_transform" /> -->
   <!--   <parent link="gripper"/> -->
   <!--   <child link="gripped_object"/> -->

Commit message: Use xacro.load_yaml to avoid warning from xacro.

File: urdf/xacro/thing_no_wheels.urdf.xacro (robot description, xacro)
@@ -35,5 +35,5 @@
   <!-- Load the base and tool transforms -->
   <xacro:property name="transform_params_file" value="$(arg transform_params)" />
-  <xacro:property name="config_transform_parameters" value="${load_yaml(transform_params_file)}"/>
+  <xacro:property name="config_transform_parameters" value="${xacro.load_yaml(transform_params_file)}"/>
   <!-- Macro to use a transform from `config_transform_parameters` as the origin. -->
   <xacro:macro name="transformed_origin" params="name">

Commit message: Add F/T sensor frame; allow home config to be specified by cmd line argument or function parameter; add parsing code for wrench messages.

File: urdf/xacro/thing_no_wheels.urdf.xacro (robot description, xacro)
@@ -231,4 +231,10 @@
     <child link="gripper"/>
   </joint>
+  <link name="ft_sensor"></link>
+  <joint name="tool_ft_sensor_joint" type="fixed">
+    <origin rpy="0 0 0" xyz="0 0 0.02"/>
+    <parent link="ur10_arm_tool0"/>
+    <child link="ft_sensor"/>
+  </joint>
   <!-- If you want to have an object as part of the URDF, include something like: -->
   <!-- <link name="gripped_object" /> -->

Commit message: Add utilities for package paths; add gripped_object to URDF by default.

File: urdf/xacro/thing_no_wheels.urdf.xacro (robot description, xacro)
@@ -237,10 +237,10 @@
     <child link="ft_sensor"/>
   </joint>
-  <!-- If you want to have an object as part of the URDF, include something like: -->
-  <!-- <link name="gripped_object" /> -->
-  <!-- <joint name="gripped_object_joint" type="fixed"> -->
-  <!--   <xacro:transformed_origin name="gripped_object_transform" /> -->
-  <!--   <parent link="gripper"/> -->
-  <!--   <child link="gripped_object"/> -->
-  <!-- </joint> -->
+  <!-- Frame for a gripped object or tool. Its pose is specified in the `transform_params` config file.  -->
+  <link name="gripped_object" />
+  <joint name="gripped_object_joint" type="fixed">
+    <xacro:transformed_origin name="gripped_object_transform" />
+    <parent link="gripper"/>
+    <child link="gripped_object"/>
+  </joint>
 </robot>

Commit message: Fix gripped_object_transform.
* Consistent naming
* Don't introduce the link in this repo; indicate dependent projects
should do that.

File: urdf/xacro/thing_no_wheels.urdf.xacro (robot description, xacro)
@@ -238,9 +238,10 @@
   </joint>
   <!-- Frame for a gripped object or tool. Its pose is specified in the `transform_params` config file.  -->
-  <link name="gripped_object" />
-  <joint name="gripped_object_joint" type="fixed">
-    <xacro:transformed_origin name="gripped_object_transform" />
-    <parent link="gripper"/>
-    <child link="gripped_object"/>
-  </joint>
+  <!-- Something like this should be added in your own project's URDF and customized to your needs. -->
+  <!-- <link name="gripped_object" /> -->
+  <!-- <joint name="gripped_object_joint" type="fixed"> -->
+  <!--   <xacro:transformed_origin name="gripped_object_transform" /> -->
+  <!--   <parent link="gripper"/> -->
+  <!--   <child link="gripped_object"/> -->
+  <!-- </joint> -->
 </robot>
