Commit message: Improve XacroDoc, use it for mm kinematics, fix offset between pybullet and pinocchio models, and add a test for this.
XacroDoc now supports making a temp file for the URDF, and has nicer
docstrings.

File: urdf/xacro/cartesian_base_joints.urdf.xacro (robot description, xacro)
@@ -37,10 +37,9 @@
     <limit effort="0.0" velocity="1000.0"/>
   </joint>
-  <!-- Note the z-offset to raise the base off the ground, to avoid collision issues. Without this, there are vibrations and other artifacts from resolving the ground collision that result in significant error in the balanced object. -->
 	<joint name="base_to_y_joint" type="continuous">
     <parent link="y_prismatic_link"/>
     <child link="base_link"/>
     <axis xyz="0 0 1"/>
-    <origin rpy="0 0 0" xyz="0 0 0.01"/>
+    <origin rpy="0 0 0" xyz="0 0 0"/>
   </joint>
 </robot>

File: urdf/xacro/thing.urdf.xacro (robot description, xacro)
@@ -1,5 +1,5 @@
 <?xml version="1.0" ?>
 <robot name="thing" xmlns:xacro="http://www.ros.org/wiki/xacro">
-  <xacro:include filename="ridgeback_wheels.urdf.xacro" />
-  <xacro:include filename="thing_no_wheels.urdf.xacro" />
+  <xacro:include filename="$(find mobile_manipulation_central)/urdf/xacro/ridgeback_wheels.urdf.xacro" />
+  <xacro:include filename="$(find mobile_manipulation_central)/urdf/xacro/thing_no_wheels.urdf.xacro" />
 </robot>

File: urdf/xacro/thing_no_wheels.urdf.xacro (robot description, xacro)
@@ -49,8 +49,15 @@
     </inertial>
   </link>
+  <!-- Note the z-offset to raise the base off the ground, to avoid collision issues in simulation. Without this, there are vibrations and other artifacts from resolving the ground collision that result in significant error in the balanced object. We include it in general for the real robot as well for consistency, to be resolved by calibration. -->
+  <joint name="dummy_base_link_joint" type="fixed">
+    <origin rpy="0 0 0" xyz="0 0 0.01"/>
+    <parent link="base_link"/>
+    <child link="dummy_base_link"/>
+  </joint>
+  <link name="dummy_base_link"/>
   <!-- Transform between base and arm can be calibrated and is loaded from parameters. -->
   <joint name="base_link_joint" type="fixed">
     <xacro:transformed_origin name="base_to_arm_transform" />
-    <parent link="base_link"/>
+    <parent link="dummy_base_link"/>
     <child link="chassis_link"/>
   </joint>

File: urdf/xacro/thing_pyb.urdf.xacro (robot description, xacro)
@@ -1,5 +1,5 @@
 <?xml version="1.0" ?>
 <robot name="thing" xmlns:xacro="http://www.ros.org/wiki/xacro">
-  <xacro:include filename="cartesian_base_joints.urdf.xacro" />
-  <xacro:include filename="thing_no_wheels.urdf.xacro" />
+  <xacro:include filename="$(find mobile_manipulation_central)/urdf/xacro/cartesian_base_joints.urdf.xacro" />
+  <xacro:include filename="$(find mobile_manipulation_central)/urdf/xacro/thing_no_wheels.urdf.xacro" />
 </robot>
